File: MCU.sch (KiCad schematic (older format))
At the start: 18 parts

Commit message: Finished schematic
Motordriver still needs footprint, it's necessary to choose new bulk capacitors
Parts:
- added R6, R7: R, Resistors_SMD:R_0402, symbol R
- C10, C11, C12, C13, C14, C15, C4, C6, C7, C8, C9: renamed from C?; footprint (none) -> Capacitors_SMD:C_0402
- C5: renamed from C?; footprint (none) -> Capacitors_SMD:C_0603
- R10, R8, R9: renamed from R?; footprint (none) -> Resistors_SMD:R_0402
- gave numbers to parts that had none: 3
Connections:
- net +3V3: now also R6.1
- net GND: now also R7.2
- net VDD_ADC: now reaches U2.10 (ADC_IN0/RTC_TAMP2/SYS_WKUP1/TIM2_CH1/TIM2_ETR/TSC_G1_IO1/USART2_CTS/PA0)
- net +5V_ADC: now reaches U2.11 (ADC_IN1/TIM2_CH2/TSC_G1_IO2/USART2_DE/USART2_RTS/PA1)
- net Current_1: now reaches U2.12 (ADC_IN2/SYS_WKUP4/TIM2_CH3/TSC_G1_IO3/USART2_TX/PA2)
- net Current_2: now reaches U2.13 (ADC_IN3/TIM2_CH4/TSC_G1_IO4/USART2_RX/PA3)
- net nFAULT_1: now reaches U2.14 (ADC_IN4/I2S1_WS/SPI1_NSS/TIM14_CH1/TSC_G2_IO1/USART2_CK/USB_OE/PA4)
- net nFAULT_2: now reaches U2.15 (ADC_IN5/CEC/I2S1_CK/SPI1_SCK/TIM2_CH1/TIM2_ETR/TSC_G2_IO2/PA5)
- net RREF_1: now reaches U2.16 (ADC_IN6/I2S1_MCK/SPI1_MISO/TIM16_CH1/TIM1_BKIN/TIM3_CH1/TSC_G2_IO3/PA6)
- net RREF_2: now reaches U2.17 (ADC_IN7/I2S1_SD/SPI1_MOSI/TIM14_CH1/TIM17_CH1/TIM1_CH1N/TIM3_CH2/TSC_G2_IO4/PA7)
- net DIR_1: now reaches U2.18 (PB0/ADC_IN8/TIM1_CH2N/TIM3_CH3/TSC_G3_IO2)
- net ENA_1: now reaches U2.19 (PB1/ADC_IN9/TIM14_CH1/TIM1_CH3N/TIM3_CH4/TSC_G3_IO3)
- net M1_1: now reaches U2.20 (PB2/TSC_G3_IO4)
- net M1_0: now reaches U2.21 (PB10/CEC/I2C1_SCL/SPI2_SCK/TIM2_CH3/TSC_SYNC)
- net nSLEEP_1: now reaches U2.22 (PB11/I2C1_SDA/TIM2_CH4)
- net TRQ_1: now reaches U2.25 (PB12/SPI2_NSS/TIM1_BKIN)
- net DECAY_1: now reaches U2.26 (PB13/I2C1_SCL/SPI2_SCK/TIM1_CH1N)
- net DECAY_2: now reaches U2.28 (PB15/RTC_REFIN/SPI2_MOSI/SYS_WKUP7/TIM1_CH3N)
- net TRQ_2: now reaches U2.29 (CRS_SYNC/RCC_MCO/TIM1_CH1/USART1_CK/PA8)
- net USART1_TX: now reaches U2.30 (I2C1_SCL/TIM1_CH2/TSC_G4_IO1/USART1_TX/PA9)
- net USART1_RX: now reaches U2.31 (I2C1_SDA/TIM17_BKIN/TIM1_CH3/TSC_G4_IO2/USART1_RX/PA10)
- net CAN_RX: now reaches U2.32 (CAN_RX/I2C1_SCL/TIM1_CH4/TSC_G4_IO3/USART1_CTS/USB_DM/PA11)
- net CAN_TX: now reaches U2.33 (CAN_TX/I2C1_SDA/TIM1_ETR/TSC_G4_IO4/USART1_DE/USART1_RTS/USB_DP/PA12)
- net CAN_S: now reaches U2.38 (I2S1_WS/SPI1_NSS/TIM2_CH1/TIM2_ETR/USART2_RX/USB_OE/PA15)
- net nSLEEP_2: now reaches U2.39 (PB3/I2S1_CK/SPI1_SCK/TIM2_CH2/TSC_G5_IO1)
- net M0_2: now reaches U2.40 (PB4/I2S1_MCK/SPI1_MISO/TIM17_BKIN/TIM3_CH1/TSC_G5_IO2)
- net M1_2: now reaches U2.41 (PB5/I2C1_SMBA/I2S1_SD/SPI1_MOSI/SYS_WKUP6/TIM16_BKIN/TIM3_CH2)
- net ENA_2: now reaches U2.42 (PB6/I2C1_SCL/TIM16_CH1N/TSC_G5_IO3/USART1_TX)
- net DIR_2: now reaches U2.43 (PB7/I2C1_SDA/TIM17_CH1N/TSC_G5_IO4/USART1_RX)
- net BOOT0: now reaches U2.44 (PF11)
- net BOOT0: now also R6.2, R7.1
- net STEP_1: now reaches U2.45 (PB8/CAN_RX/CEC/I2C1_SCL/TIM16_CH1/TSC_SYNC)
- net STEP_2: now reaches U2.46 (PB9/CAN_TX/I2C1_SDA/IR_OUT/SPI2_NSS/TIM17_CH1)
- no-connect marks 1 -> 5
Other:
- note added: "Update CubeMX file when changing Pinout!!!"

Commit message: small updates
Other:
- note added: "CubeMX shows which pins can be remapped\nwithout effecting functionality.\n\nThey are "unpinned" in the design.\nUpdate CubeMX file after changing Pinout!!!"
- note removed: "Update CubeMX file when changing Pinout!!!"
- moved on the sheet: C10, C12, C14, C15

Commit message: udated schematics
Parts:
- C5: value >1uF 16V -> 10uF 16V
- R6: value R -> NM
- R7: value R -> 10K
- R9: value R -> 4R7
Changed lines of the file:
@@
 $EndComp
 $Comp
-L GND #PWR025
+L GND #PWR27
 U 1 1 5A088CC4
 P 2050 3700
-F 0 "#PWR025" H 2050 3450 50  0001 C CNN
+F 0 "#PWR27" H 2050 3450 50  0001 C CNN
 F 1 "GND" H 2050 3550 50  0000 C CNN
 F 2 "" H 2050 3700 50  0001 C CNN
@@
 $EndComp
 $Comp
-L GND #PWR026
+L GND #PWR29
 U 1 1 5A088CE5
 P 2350 3700
-F 0 "#PWR026" H 2350 3450 50  0001 C CNN
+F 0 "#PWR29" H 2350 3450 50  0001 C CNN
 F 1 "GND" H 2350 3550 50  0000 C CNN
 F 2 "" H 2350 3700 50  0001 C CNN
@@
 $EndComp
 $Comp
-L GND #PWR027
+L GND #PWR24
 U 1 1 5A088CFF
 P 1700 3700
-F 0 "#PWR027" H 1700 3450 50  0001 C CNN
+F 0 "#PWR24" H 1700 3450 50  0001 C CNN
 F 1 "GND" H 1700 3550 50  0000 C CNN
 F 2 "" H 1700 3700 50  0001 C CNN
@@
 $EndComp
 $Comp
-L GND #PWR028
+L GND #PWR31
 U 1 1 5A088E51
 P 2950 2750
-F 0 "#PWR028" H 2950 2500 50  0001 C CNN
+F 0 "#PWR31" H 2950 2500 50  0001 C CNN
 F 1 "GND" H 2950 2600 50  0000 C CNN
 F 2 "" H 2950 2750 50  0001 C CNN
@@
 $EndComp
 $Comp
-L +3V3 #PWR029
+L +3V3 #PWR35
 U 1 1 5A0893C3
 P 4100 1250
-F 0 "#PWR029" H 4100 1100 50  0001 C CNN
+F 0 "#PWR35" H 4100 1100 50  0001 C CNN
 F 1 "+3V3" H 4100 1390 50  0000 C CNN
 F 2 "" H 4100 1250 50  0001 C CNN
@@
 $EndComp
 $Comp
-L GND #PWR030
+L GND #PWR36
 U 1 1 5A08949D
 P 4100 1650
-F 0 "#PWR030" H 4100 1400 50  0001 C CNN
+F 0 "#PWR36" H 4100 1400 50  0001 C CNN
 F 1 "GND" H 4100 1500 50  0000 C CNN
 F 2 "" H 4100 1650 50  0001 C CNN
@@
 $EndComp
 $Comp
-L +3V3 #PWR031
+L +3V3 #PWR47
 U 1 1 5A089891
 P 6250 2050
-F 0 "#PWR031" H 6250 1900 50  0001 C CNN
+F 0 "#PWR47" H 6250 1900 50  0001 C CNN
 F 1 "+3V3" H 6250 2190 50  0000 C CNN
 F 2 "" H 6250 2050 50  0001 C CNN
@@
 $EndComp
 $Comp
-L GND #PWR032
+L GND #PWR48
 U 1 1 5A089D57
 P 6250 5950
-F 0 "#PWR032" H 6250 5700 50  0001 C CNN
+F 0 "#PWR48" H 6250 5700 50  0001 C CNN
 F 1 "GND" H 6250 5800 50  0000 C CNN
 F 2 "" H 6250 5950 50  0001 C CNN
@@
 $EndComp
 $Comp
-L +3V3 #PWR033
+L +3V3 #PWR37
 U 1 1 5A08B29F
 P 4500 1250
-F 0 "#PWR033" H 4500 1100 50  0001 C CNN
+F 0 "#PWR37" H 4500 1100 50  0001 C CNN
 F 1 "+3V3" H 4500 1390 50  0000 C CNN
 F 2 "" H 4500 1250 50  0001 C CNN
@@
 $EndComp
 $Comp
-L GND #PWR034
+L GND #PWR38
 U 1 1 5A08B2A5
 P 4500 1650
-F 0 "#PWR034" H 4500 1400 50  0001 C CNN
+F 0 "#PWR38" H 4500 1400 50  0001 C CNN
 F 1 "GND" H 4500 1500 50  0000 C CNN
 F 2 "" H 4500 1650 50  0001 C CNN
@@
 $EndComp
 $Comp
-L +3V3 #PWR035
+L +3V3 #PWR39
 U 1 1 5A08B2D8
 P 4900 1250
-F 0 "#PWR035" H 4900 1100 50  0001 C CNN
+F 0 "#PWR39" H 4900 1100 50  0001 C CNN
 F 1 "+3V3" H 4900 1390 50  0000 C CNN
 F 2 "" H 4900 1250 50  0001 C CNN
@@
 $EndComp
 $Comp
-L GND #PWR036
+L GND #PWR40
 U 1 1 5A08B2DE
 P 4900 1650
-F 0 "#PWR036" H 4900 1400 50  0001 C CNN
+F 0 "#PWR40" H 4900 1400 50  0001 C CNN
 F 1 "GND" H 4900 1500 50  0000 C CNN
 F 2 "" H 4900 1650 50  0001 C CNN
@@
 $EndComp
 $Comp
-L +3V3 #PWR037
+L +3V3 #PWR41
 U 1 1 5A08B322
 P 5300 1250
-F 0 "#PWR037" H 5300 1100 50  0001 C CNN
+F 0 "#PWR41" H 5300 1100 50  0001 C CNN
 F 1 "+3V3" H 5300 1390 50  0000 C CNN
 F 2 "" H 5300 1250 50  0001 C CNN
@@
 $EndComp
 $Comp
-L GND #PWR038
+L GND #PWR42
 U 1 1 5A08B328
 P 5300 1650
-F 0 "#PWR038" H 5300 1400 50  0001 C CNN
+F 0 "#PWR42" H 5300 1400 50  0001 C CNN
 F 1 "GND" H 5300 1500 50  0000 C CNN
 F 2 "" H 5300 1650 50  0001 C CNN
@@
 $EndComp
 $Comp
-L +3V3 #PWR039
+L +3V3 #PWR43
 U 1 1 5A08B36E
 P 5700 1250
-F 0 "#PWR039" H 5700 1100 50  0001 C CNN
+F 0 "#PWR43" H 5700 1100 50  0001 C CNN
 F 1 "+3V3" H 5700 1390 50  0000 C CNN
 F 2 "" H 5700 1250 50  0001 C CNN
@@
 $EndComp
 $Comp
-L GND #PWR040
+L GND #PWR44
 U 1 1 5A08B374
 P 5700 1650
-F 0 "#PWR040" H 5700 1400 50  0001 C CNN
+F 0 "#PWR44" H 5700 1400 50  0001 C CNN
 F 1 "GND" H 5700 1500 50  0000 C CNN
 F 2 "" H 5700 1650 50  0001 C CNN
@@
 P 1850 6500
 F 0 "R9" V 1930 6500 50  0000 C CNN
-F 1 "R" V 1850 6500 50  0000 C CNN
+F 1 "4R7" V 1850 6500 50  0000 C CNN
 F 2 "Resistors_SMD:R_0402" V 1780 6500 50  0001 C CNN
 F 3 "" H 1850 6500 50  0001 C CNN
@@
 P 2300 6800
 F 0 "C5" H 2325 6900 50  0000 L CNN
-F 1 ">1uF 16V" V 2150 6650 50  0000 L CNN
+F 1 "10uF 16V" V 2150 6650 50  0000 L CNN
 F 2 "Capacitors_SMD:C_0603" H 2338 6650 50  0001 C CNN
 F 3 "" H 2300 6800 50  0001 C CNN
@@
 $EndComp
 $Comp
-L GND #PWR041
+L GND #PWR28
 U 1 1 5A16E036
 P 2300 7000
-F 0 "#PWR041" H 2300 6750 50  0001 C CNN
+F 0 "#PWR28" H 2300 6750 50  0001 C CNN
 F 1 "GND" H 2300 6850 50  0000 C CNN
 F 2 "" H 2300 7000 50  0001 C CNN
@@
 $EndComp
 $Comp
-L GND #PWR042
+L GND #PWR30
 U 1 1 5A16E0FE
 P 2850 7000
-F 0 "#PWR042" H 2850 6750 50  0001 C CNN
+F 0 "#PWR30" H 2850 6750 50  0001 C CNN
 F 1 "GND" H 2850 6850 50  0000 C CNN
 F 2 "" H 2850 7000 50  0001 C CNN
@@
 $EndComp
 $Comp
-L VDD #PWR043
+L VDD #PWR23
 U 1 1 5A16E437
 P 1650 6200
-F 0 "#PWR043" H 1650 6050 50  0001 C CNN
+F 0 "#PWR23" H 1650 6050 50  0001 C CNN
 F 1 "VDD" H 1650 6350 50  0000 C CNN
 F 2 "" H 1650 6200 50  0001 C CNN
@@
 $EndComp
 $Comp
-L +5V #PWR044
+L +5V #PWR22
 U 1 1 5A16E4D9
 P 1400 6200
-F 0 "#PWR044" H 1400 6050 50  0001 C CNN
+F 0 "#PWR22" H 1400 6050 50  0001 C CNN
 F 1 "+5V" H 1400 6340 50  0000 C CNN
 F 2 "" H 1400 6200 50  0001 C CNN
@@
 $EndComp
 $Comp
-L GND #PWR045
+L GND #PWR32
 U 1 1 5A16ED6D
 P 3450 7000
-F 0 "#PWR045" H 3450 6750 50  0001 C CNN
+F 0 "#PWR32" H 3450 6750 50  0001 C CNN
 F 1 "GND" H 3450 6850 50  0000 C CNN
 F 2 "" H 3450 7000 50  0001 C CNN
@@
 $EndComp
 $Comp
-L GND #PWR046
+L GND #PWR34
 U 1 1 5A16F0D6
 P 3800 7000
-F 0 "#PWR046" H 3800 6750 50  0001 C CNN
+F 0 "#PWR34" H 3800 6750 50  0001 C CNN
 F 1 "GND" H 3800 6850 50  0000 C CNN
 F 2 "" H 3800 7000 50  0001 C CNN
@@
 $EndComp
 $Comp
-L +3V3 #PWR047
+L +3V3 #PWR33
 U 1 1 5A16F152
 P 3800 6400
-F 0 "#PWR047" H 3800 6250 50  0001 C CNN
+F 0 "#PWR33" H 3800 6250 50  0001 C CNN
 F 1 "+3V3" H 3800 6540 50  0000 C CNN
 F 2 "" H 3800 6400 50  0001 C CNN
@@
 $EndComp
 $Comp
-L +3V3 #PWR048
+L +3V3 #PWR45
 U 1 1 5A171D39
 P 6100 1250
-F 0 "#PWR048" H 6100 1100 50  0001 C CNN
+F 0 "#PWR45" H 6100 1100 50  0001 C CNN
 F 1 "+3V3" H 6100 1390 50  0000 C CNN
 F 2 "" H 6100 1250 50  0001 C CNN
@@
 $EndComp
 $Comp
-L GND #PWR049
+L GND #PWR46
 U 1 1 5A171D3F
 P 6100 1650
-F 0 "#PWR049" H 6100 1400 50  0001 C CNN
+F 0 "#PWR46" H 6100 1400 50  0001 C CNN
 F 1 "GND" H 6100 1500 50  0000 C CNN
 F 2 "" H 6100 1650 50  0001 C CNN
@@
 P 1800 1400
 F 0 "R6" V 1880 1400 50  0000 C CNN
-F 1 "R" V 1800 1400 50  0000 C CNN
+F 1 "NM" V 1800 1400 50  0000 C CNN
 F 2 "Resistors_SMD:R_0402" V 1730 1400 50  0001 C CNN
 F 3 "" H 1800 1400 50  0001 C CNN
@@
 P 1800 1800
 F 0 "R7" V 1880 1800 50  0000 C CNN
-F 1 "R" V 1800 1800 50  0000 C CNN
+F 1 "10K" V 1800 1800 50  0000 C CNN
 F 2 "Resistors_SMD:R_0402" V 1730 1800 50  0001 C CNN
 F 3 "" H 1800 1800 50  0001 C CNN
@@
 	1800 1550 1800 1650
 $Comp
-L GND #PWR050
+L GND #PWR26
 U 1 1 5A1F759D
 P 1800 2000
-F 0 "#PWR050" H 1800 1750 50  0001 C CNN
+F 0 "#PWR26" H 1800 1750 50  0001 C CNN
 F 1 "GND" H 1800 1850 50  0000 C CNN
 F 2 "" H 1800 2000 50  0001 C CNN
@@
 	1800 1950 1800 2000
 $Comp
-L +3V3 #PWR051
+L +3V3 #PWR25
 U 1 1 5A1F76F4
 P 1800 1200
-F 0 "#PWR051" H 1800 1050 50  0001 C CNN
+F 0 "#PWR25" H 1800 1050 50  0001 C CNN
 F 1 "+3V3" H 1800 1340 50  0000 C CNN
 F 2 "" H 1800 1200 50  0001 C CNN
@@
 Connection ~ 1800 1600
 $Comp
-L PWR_FLAG #FLG052
+L PWR_FLAG #FLG4
 U 1 1 5A2027E3
 P 2300 6200
-F 0 "#FLG052" H 2300 6275 50  0001 C CNN
+F 0 "#FLG4" H 2300 6275 50  0001 C CNN
 F 1 "PWR_FLAG" H 2300 6350 50  0000 C CNN
 F 2 "" H 2300 6200 50  0001 C CNN

Commit message: started modifying for 3 stepper motors
Connections:
- net Current_2 is gone; now on net nFAULT_1: U2.13 (ADC_IN3/TIM2_CH4/TSC_G1_IO4/USART2_RX/PA3)
- net nFAULT_1: no longer U2.14 (ADC_IN4/I2S1_WS/SPI1_NSS/TIM14_CH1/TSC_G2_IO1/USART2_CK/USB_OE/PA4)
- net nFAULT_2: now also U2.2 (PC13/RTC_OUT_ALARM/RTC_OUT_CALIB/RTC_TAMP1/RTC_TS/SYS_WKUP2); no longer U2.15 (ADC_IN5/CEC/I2S1_CK/SPI1_SCK/TIM2_CH1/TIM2_ETR/TSC_G2_IO2/PA5)
- net CAN_S: no longer names the net of U2.38 (I2S1_WS/SPI1_NSS/TIM2_CH1/TIM2_ETR/USART2_RX/USB_OE/PA15)
- net Current_1 renamed Current
- net ENA_1 renamed ENA
- net ENA_2: no longer names the net of U2.42 (PB6/I2C1_SCL/TIM16_CH1N/TSC_G5_IO3/USART1_TX)
- net nSLEEP_1 renamed nSLEEP
- net nSLEEP_2: no longer names the net of U2.39 (PB3/I2S1_CK/SPI1_SCK/TIM2_CH2/TSC_G5_IO1)
- new net STEP_3: U2.14 (ADC_IN4/I2S1_WS/SPI1_NSS/TIM14_CH1/TSC_G2_IO1/USART2_CK/USB_OE/PA4)
- new net nFAULT_3: U2.15 (ADC_IN5/CEC/I2S1_CK/SPI1_SCK/TIM2_CH1/TIM2_ETR/TSC_G2_IO2/PA5)
- no-connect marks 5 -> 1
Changed lines of the file:
@@
 $Descr A4 11693 8268
 encoding utf-8
-Sheet 2 4
+Sheet 4 4
 Title ""
 Date ""
@@
 +5V_ADC
 Text HLabel 9650 4100 2    60   Input ~ 0
-Current_1
-Text HLabel 9650 4200 2    60   Input ~ 0
-Current_2
+Current
 Text HLabel 9650 5100 2    60   Output ~ 0
 CAN_TX
@@
 	9550 4100 9650 4100
 Wire Wire Line
-	9650 4200 9550 4200
-Wire Wire Line
 	9550 4900 9650 4900
 Wire Wire Line
@@
 Wire Wire Line
 	2350 3300 2350 3200
-Text HLabel 9650 5400 2    60   Output ~ 0
-CAN_S
-Wire Wire Line
-	9550 5400 9650 5400
-Text HLabel 9650 4300 2    60   Input ~ 0
+Text HLabel 9650 4200 2    60   Input ~ 0
 nFAULT_1
-Text HLabel 9650 4400 2    60   Input ~ 0
-nFAULT_2
 Wire Wire Line
 	9650 4300 9550 4300
@@
 	3250 3900 3350 3900
 Text HLabel 3250 4000 0    60   Output ~ 0
-ENA_1
+ENA
 Text HLabel 3250 4100 0    60   Output ~ 0
 M1_1
@@
 Wire Wire Line
 	3250 4900 3350 4900
-Text HLabel 3250 5000 0    60   Output ~ 0
-nSLEEP_1
 Wire Wire Line
 	3250 5000 3350 5000
@@
 Text HLabel 3250 5200 0    60   Output ~ 0
 DECAY_1
-NoConn ~ 3350 5300
 Text HLabel 3250 5400 0    60   Output ~ 0
 DECAY_2
@@
 Wire Wire Line
 	3250 4000 3350 4000
-Text HLabel 3250 4200 0    60   Output ~ 0
-nSLEEP_2
 Text HLabel 3250 4300 0    60   Output ~ 0
 M0_2
 Text HLabel 3250 4400 0    60   Output ~ 0
 M1_2
-Text HLabel 3250 4500 0    60   Output ~ 0
-ENA_2
 Text HLabel 3250 4600 0    60   Output ~ 0
 DIR_2
@@
 	3350 4600 3250 4600
 Wire Wire Line
-	3250 4500 3350 4500
-Wire Wire Line
 	3250 4400 3350 4400
 Wire Wire Line
 	3250 4300 3350 4300
-Wire Wire Line
-	3250 4200 3350 4200
-NoConn ~ 3350 3500
-NoConn ~ 3350 3600
-NoConn ~ 3350 3700
 Text Label 3250 3300 2    60   ~ 0
 BOOT0
@@
 Text Notes 600  4650 0    60   ~ 0
 CubeMX shows which pins can be remapped\nwithout effecting functionality.\n\nThey are "unpinned" in the design.\nUpdate CubeMX file after changing Pinout!!!
+Text HLabel 3250 5000 0    60   Output ~ 0
+nSLEEP
+Text HLabel 9650 4400 2    60   Input ~ 0
+nFAULT_3
+Wire Wire Line
+	9650 4200 9550 4200
+Text HLabel 3250 3500 0    60   Input ~ 0
+nFAULT_2
+Wire Wire Line
+	3250 3500 3350 3500
+Text HLabel 9650 4300 2    60   Output ~ 0
+STEP_3
 $EndSCHEMATC
