File: Mot_driver.sch (KiCad schematic (older format))
At the start: 36 parts

Commit message: Finished schematic
Motordriver still needs footprint, it's necessary to choose new bulk capacitors
Parts:
- C16, C28: renamed from C?; footprint (none) -> Capacitors_SMD:C_1206
- C17, C18, C19, C20, C21, C22, C23, C24, C25, C26, C27, C29, C30, C31, C32, C33, C34, C35: renamed from C?; footprint (none) -> Capacitors_SMD:C_0402
- R11, R17: renamed from R?; footprint (none) -> lakotamm-shunt:R_0603
- R12, R13, R14, R15, R16, R18, R19, R20, R21, R22: renamed from R?; footprint (none) -> Resistors_SMD:R_0402
- gave numbers to parts that had none: 4
Connections:
- net nFAULT renamed nFAULT_1
- net nFAULT_1: no longer U6.15 (nFAULT)
- net nSLEEP renamed nSLEEP_1
- net nSLEEP_1: no longer U6.17 (nSLEEP)
- new net nFAULT_2: U6.15 (nFAULT)
- new net nSLEEP_2: U6.17 (nSLEEP)

Commit message: small updates
Parts:
- U4, U6: footprint (none) -> lakotamm-motordriver:TSSOP-24_1E_4.4x7.8mm_Pitch0.65mm
Connections:
- net GND: now also U4.25 (Thermal_pad), U6.25 (Thermal_pad)
Changed lines of the file:
@@
 F 0 "U4" H 3900 450 60  0000 C CNN
 F 1 "DRV8886AT" H 3300 450 60  0000 C CNN
-F 2 "" H 3750 850 60  0001 C CNN
+F 2 "lakotamm-motordriver:TSSOP-24_1E_4.4x7.8mm_Pitch0.65mm" H 3750 850 60  0001 C CNN
 F 3 "http://www.ti.com/lit/ds/symlink/drv8886at.pdf" H 3500 850 60  0001 C CNN
 F 4 "DRV8886ATPWP" H 3500 3650 60  0001 C CNN "MPN"
@@
 $EndComp
 $Comp
-L GND #PWR53
+L GND #PWR053
 U 1 1 5A114125
 P 1950 1600
-F 0 "#PWR53" H 1950 1350 50  0001 C CNN
+F 0 "#PWR053" H 1950 1350 50  0001 C CNN
 F 1 "GND" H 1950 1450 50  0000 C CNN
 F 2 "" H 1950 1600 50  0001 C CNN
@@
 $EndComp
 $Comp
-L GND #PWR57
+L GND #PWR054
 U 1 1 5A114140
 P 2300 1600
-F 0 "#PWR57" H 2300 1350 50  0001 C CNN
+F 0 "#PWR054" H 2300 1350 50  0001 C CNN
 F 1 "GND" H 2300 1450 50  0000 C CNN
 F 2 "" H 2300 1600 50  0001 C CNN
@@
 $EndComp
 $Comp
-L GND #PWR52
+L GND #PWR055
 U 1 1 5A115586
 P 1850 2850
-F 0 "#PWR52" H 1850 2600 50  0001 C CNN
+F 0 "#PWR055" H 1850 2600 50  0001 C CNN
 F 1 "GND" H 1850 2700 50  0000 C CNN
 F 2 "" H 1850 2850 50  0001 C CNN
@@
 $EndComp
 $Comp
-L GND #PWR56
+L GND #PWR056
 U 1 1 5A11659E
 P 2200 2850
-F 0 "#PWR56" H 2200 2600 50  0001 C CNN
+F 0 "#PWR056" H 2200 2600 50  0001 C CNN
 F 1 "GND" H 2200 2700 50  0000 C CNN
 F 2 "" H 2200 2850 50  0001 C CNN
@@
 $EndComp
 $Comp
-L GND #PWR60
+L GND #PWR057
 U 1 1 5A11673F
 P 2700 2650
-F 0 "#PWR60" H 2700 2400 50  0001 C CNN
+F 0 "#PWR057" H 2700 2400 50  0001 C CNN
 F 1 "GND" H 2850 2650 50  0000 C CNN
 F 2 "" H 2700 2650 50  0001 C CNN
@@
 TRQ_1
 $Comp
-L GND #PWR63
+L GND #PWR058
 U 1 1 5A117564
 P 4250 2100
-F 0 "#PWR63" H 4250 1850 50  0001 C CNN
+F 0 "#PWR058" H 4250 1850 50  0001 C CNN
 F 1 "GND" H 4100 2050 50  0000 C CNN
 F 2 "" H 4250 2100 50  0001 C CNN
@@
 $EndComp
 $Comp
-L GND #PWR64
+L GND #PWR059
 U 1 1 5A11794A
 P 4250 3600
-F 0 "#PWR64" H 4250 3350 50  0001 C CNN
+F 0 "#PWR059" H 4250 3350 50  0001 C CNN
 F 1 "GND" H 4100 3550 50  0000 C CNN
 F 2 "" H 4250 3600 50  0001 C CNN
@@
 $EndComp
 $Comp
-L GND #PWR61
+L GND #PWR060
 U 1 1 5A1210B8
 P 2700 4850
-F 0 "#PWR61" H 2700 4600 50  0001 C CNN
+F 0 "#PWR060" H 2700 4600 50  0001 C CNN
 F 1 "GND" H 2700 4700 50  0000 C CNN
 F 2 "" H 2700 4850 50  0001 C CNN
@@
 $EndComp
 $Comp
-L GND #PWR51
+L GND #PWR061
 U 1 1 5A12197F
 P 1700 4500
-F 0 "#PWR51" H 1700 4250 50  0001 C CNN
+F 0 "#PWR061" H 1700 4250 50  0001 C CNN
 F 1 "GND" H 1700 4350 50  0000 C CNN
 F 2 "" H 1700 4500 50  0001 C CNN
@@
 $EndComp
 $Comp
-L GND #PWR58
+L GND #PWR062
 U 1 1 5A121EB9
 P 2350 4850
-F 0 "#PWR58" H 2350 4600 50  0001 C CNN
+F 0 "#PWR062" H 2350 4600 50  0001 C CNN
 F 1 "GND" H 2350 4700 50  0000 C CNN
 F 2 "" H 2350 4850 50  0001 C CNN
@@
 F 0 "U6" H 8200 450 60  0000 C CNN
 F 1 "DRV8886AT" H 7600 450 60  0000 C CNN
-F 2 "" H 8050 850 60  0001 C CNN
+F 2 "lakotamm-motordriver:TSSOP-24_1E_4.4x7.8mm_Pitch0.65mm" H 8050 850 60  0001 C CNN
 F 3 "http://www.ti.com/lit/ds/symlink/drv8886at.pdf" H 7800 850 60  0001 C CNN
 F 4 "DRV8886ATPWP" H 7800 3650 60  0001 C CNN "MPN"
@@
 $EndComp
 $Comp
-L GND #PWR73
+L GND #PWR063
 U 1 1 5A123A44
 P 6250 1600
-F 0 "#PWR73" H 6250 1350 50  0001 C CNN
+F 0 "#PWR063" H 6250 1350 50  0001 C CNN
 F 1 "GND" H 6250 1450 50  0000 C CNN
 F 2 "" H 6250 1600 50  0001 C CNN
@@
 $EndComp
 $Comp
-L GND #PWR75
+L GND #PWR064
 U 1 1 5A123A4A
 P 6600 1600
-F 0 "#PWR75" H 6600 1350 50  0001 C CNN
+F 0 "#PWR064" H 6600 1350 50  0001 C CNN
 F 1 "GND" H 6600 1450 50  0000 C CNN
 F 2 "" H 6600 1600 50  0001 C CNN
@@
 $EndComp
 $Comp
-L GND #PWR72
+L GND #PWR065
 U 1 1 5A123A59
 P 6150 2850
-F 0 "#PWR72" H 6150 2600 50  0001 C CNN
+F 0 "#PWR065" H 6150 2600 50  0001 C CNN
 F 1 "GND" H 6150 2700 50  0000 C CNN
 F 2 "" H 6150 2850 50  0001 C CNN
@@
 $EndComp
 $Comp
-L GND #PWR74
+L GND #PWR066
 U 1 1 5A123A79
 P 6500 2850
-F 0 "#PWR74" H 6500 2600 50  0001 C CNN
+F 0 "#PWR066" H 6500 2600 50  0001 C CNN
 F 1 "GND" H 6500 2700 50  0000 C CNN
 F 2 "" H 6500 2850 50  0001 C CNN
@@
 $EndComp
 $Comp
-L GND #PWR77
+L GND #PWR067
 U 1 1 5A123A8A
 P 7000 2650
-F 0 "#PWR77" H 7000 2400 50  0001 C CNN
+F 0 "#PWR067" H 7000 2400 50  0001 C CNN
 F 1 "GND" H 7150 2650 50  0000 C CNN
 F 2 "" H 7000 2650 50  0001 C CNN
@@
 TRQ_2
 $Comp
-L VDD #PWR67
+L VDD #PWR068
 U 1 1 5A123AA0
 P 5200 1050
-F 0 "#PWR67" H 5200 900 50  0001 C CNN
+F 0 "#PWR068" H 5200 900 50  0001 C CNN
 F 1 "VDD" H 5200 1200 50  0000 C CNN
 F 2 "" H 5200 1050 50  0001 C CNN
@@
 $EndComp
 $Comp
-L GND #PWR79
+L GND #PWR069
 U 1 1 5A123AA7
 P 8550 2100
-F 0 "#PWR79" H 8550 1850 50  0001 C CNN
+F 0 "#PWR069" H 8550 1850 50  0001 C CNN
 F 1 "GND" H 8400 2050 50  0000 C CNN
 F 2 "" H 8550 2100 50  0001 C CNN
@@
 $EndComp
 $Comp
-L GND #PWR80
+L GND #PWR070
 U 1 1 5A123AAF
 P 8550 3600
-F 0 "#PWR80" H 8550 3350 50  0001 C CNN
+F 0 "#PWR070" H 8550 3350 50  0001 C CNN
 F 1 "GND" H 8400 3550 50  0000 C CNN
 F 2 "" H 8550 3600 50  0001 C CNN
@@
 $EndComp
 $Comp
-L GND #PWR78
+L GND #PWR071
 U 1 1 5A123AC7
 P 7000 4850
-F 0 "#PWR78" H 7000 4600 50  0001 C CNN
+F 0 "#PWR071" H 7000 4600 50  0001 C CNN
 F 1 "GND" H 7000 4700 50  0000 C CNN
 F 2 "" H 7000 4850 50  0001 C CNN
@@
 $EndComp
 $Comp
-L GND #PWR71
+L GND #PWR072
 U 1 1 5A123AD4
 P 6000 4500
-F 0 "#PWR71" H 6000 4250 50  0001 C CNN
+F 0 "#PWR072" H 6000 4250 50  0001 C CNN
 F 1 "GND" H 6000 4350 50  0000 C CNN
 F 2 "" H 6000 4500 50  0001 C CNN
@@
 $EndComp
 $Comp
-L GND #PWR76
+L GND #PWR073
 U 1 1 5A123AED
 P 6650 4850
-F 0 "#PWR76" H 6650 4600 50  0001 C CNN
+F 0 "#PWR073" H 6650 4600 50  0001 C CNN
 F 1 "GND" H 6650 4700 50  0000 C CNN
 F 2 "" H 6650 4850 50  0001 C CNN
@@
 $EndComp
 $Comp
-L GND #PWR70
+L GND #PWR074
 U 1 1 5A125921
 P 5900 1600
-F 0 "#PWR70" H 5900 1350 50  0001 C CNN
+F 0 "#PWR074" H 5900 1350 50  0001 C CNN
 F 1 "GND" H 5900 1450 50  0000 C CNN
 F 2 "" H 5900 1600 50  0001 C CNN
@@
 $EndComp
 $Comp
-L GND #PWR50
+L GND #PWR075
 U 1 1 5A125AA7
 P 1600 1600
-F 0 "#PWR50" H 1600 1350 50  0001 C CNN
+F 0 "#PWR075" H 1600 1350 50  0001 C CNN
 F 1 "GND" H 1600 1450 50  0000 C CNN
 F 2 "" H 1600 1600 50  0001 C CNN
@@
 SH2-
 $Comp
-L VDD #PWR49
+L VDD #PWR076
 U 1 1 5A14752A
 P 900 1050
-F 0 "#PWR49" H 900 900 50  0001 C CNN
+F 0 "#PWR076" H 900 900 50  0001 C CNN
 F 1 "VDD" H 900 1200 50  0000 C CNN
 F 2 "" H 900 1050 50  0001 C CNN
@@
 $EndComp
 $Comp
-L GND #PWR55
+L GND #PWR077
 U 1 1 5A154EFF
 P 2100 6900
-F 0 "#PWR55" H 2100 6650 50  0001 C CNN
+F 0 "#PWR077" H 2100 6650 50  0001 C CNN
 F 1 "GND" H 2100 6750 50  0000 C CNN
 F 2 "" H 2100 6900 50  0001 C CNN
@@
 $EndComp
 $Comp
-L +3V3 #PWR54
+L +3V3 #PWR078
 U 1 1 5A155966
 P 2100 5750
-F 0 "#PWR54" H 2100 5600 50  0001 C CNN
+F 0 "#PWR078" H 2100 5600 50  0001 C CNN
 F 1 "+3V3" H 2100 5890 50  0000 C CNN
 F 2 "" H 2100 5750 50  0001 C CNN
@@
 $EndComp
 $Comp
-L GND #PWR59
+L GND #PWR079
 U 1 1 5A155EC9
 P 2550 6050
-F 0 "#PWR59" H 2550 5800 50  0001 C CNN
+F 0 "#PWR079" H 2550 5800 50  0001 C CNN
 F 1 "GND" H 2550 5900 50  0000 C CNN
 F 2 "" H 2550 6050 50  0001 C CNN
@@
 $EndComp
 $Comp
-L GND #PWR62
+L GND #PWR080
 U 1 1 5A157485
 P 3150 6900
-F 0 "#PWR62" H 3150 6650 50  0001 C CNN
+F 0 "#PWR080" H 3150 6650 50  0001 C CNN
 F 1 "GND" H 3150 6750 50  0000 C CNN
 F 2 "" H 3150 6900 50  0001 C CNN
@@
 $EndComp
 $Comp
-L GND #PWR66
+L GND #PWR081
 U 1 1 5A15A10A
 P 4800 6950
-F 0 "#PWR66" H 4800 6700 50  0001 C CNN
+F 0 "#PWR081" H 4800 6700 50  0001 C CNN
 F 1 "GND" H 4800 6800 50  0000 C CNN
 F 2 "" H 4800 6950 50  0001 C CNN
@@
 $EndComp
 $Comp
-L +3V3 #PWR65
+L +3V3 #PWR082
 U 1 1 5A15A110
 P 4800 5800
-F 0 "#PWR65" H 4800 5650 50  0001 C CNN
+F 0 "#PWR082" H 4800 5650 50  0001 C CNN
 F 1 "+3V3" H 4800 5940 50  0000 C CNN
 F 2 "" H 4800 5800 50  0001 C CNN
@@
 $EndComp
 $Comp
-L GND #PWR68
+L GND #PWR083
 U 1 1 5A15A11C
 P 5250 6100
-F 0 "#PWR68" H 5250 5850 50  0001 C CNN
+F 0 "#PWR083" H 5250 5850 50  0001 C CNN
 F 1 "GND" H 5250 5950 50  0000 C CNN
 F 2 "" H 5250 6100 50  0001 C CNN
@@
 $EndComp
 $Comp
-L GND #PWR69
+L GND #PWR084
 U 1 1 5A15A128
 P 5850 6950
-F 0 "#PWR69" H 5850 6700 50  0001 C CNN
+F 0 "#PWR084" H 5850 6700 50  0001 C CNN
 F 1 "GND" H 5850 6800 50  0000 C CNN
 F 2 "" H 5850 6950 50  0001 C CNN
@@
 	4300 6250 4300 6350
 Connection ~ 4300 6350
+$Comp
+L GND #PWR085
+U 1 1 5A14EDEC
+P 8550 4100
+F 0 "#PWR085" H 8550 3850 50  0001 C CNN
+F 1 "GND" H 8400 4050 50  0000 C CNN
+F 2 "" H 8550 4100 50  0001 C CNN
+F 3 "" H 8550 4100 50  0001 C CNN
+	1    8550 4100
+	1    0    0    -1
+$EndComp
+Wire Wire Line
+	8450 4050 8550 4050
+Wire Wire Line
+	8550 4050 8550 4100
+$Comp
+L GND #PWR086
+U 1 1 5A14EF33
+P 4250 4100
+F 0 "#PWR086" H 4250 3850 50  0001 C CNN
+F 1 "GND" H 4100 4050 50  0000 C CNN
+F 2 "" H 4250 4100 50  0001 C CNN
+F 3 "" H 4250 4100 50  0001 C CNN
+	1    4250 4100
+	1    0    0    -1
+$EndComp
+Wire Wire Line
+	4150 4050 4250 4050
+Wire Wire Line
+	4250 4050 4250 4100
 $EndSCHEMATC

Commit message: udated schematics
Parts:
- added R12, R20: 0R, Resistors_SMD:R_0402, symbol R
- C16, C28: value C -> 47u 16V; MPN (none) -> GRM31CR61C476ME44
- C22, C33: value C -> 1u 6V3
- R11: value R_Shunt -> R022
- R13: renamed from R12; value R -> NM
- R14: renamed from R13; value R -> 36k
- R15: renamed from R14; value R -> 20k
- R16: renamed from R15; value R -> 20k
- R17: renamed from R16; value R -> 1k
- R18: renamed from R17; value R_Shunt -> R022
- R19: renamed from R18; value R -> 1k
- R21: renamed from R19; value R -> NM
- R22: renamed from R20; value R -> 36k
- R23: renamed from R21; value R -> 20k
- R24: renamed from R22; value R -> 20k
- U3, U5: value INA199 -> INA199A2
Connections:
- net +3V3: now also R12.1, R20.1
- net DECAY_1: now also R12.2
- net DECAY_2: now also R20.2
Other:
- note added: "There values allow the MCU to adjust output current between (almost) 0 and 0,915A"
- moved on the sheet: C17, C29, R13, R21

Commit message: started modifying for 3 stepper motors
Parts:
- removed C21, C26: 100n 6V3, Capacitors_SMD:C_0402, symbol C
- removed C25, C27: 1u 6V3, Capacitors_SMD:C_0402, symbol C
- removed R11, R18: R022, lakotamm-shunt:R_0603, symbol R_Shunt
- removed R17, R19: 1k, Resistors_SMD:R_0402, symbol R
- removed U3, U5: INA199A2, Housings_DFN_QFN:UQFN-10_1.4x1.8mm_Pitch0.4mm, symbol INA199
- added C? (x2): 10n 16V, Capacitors_SMD:C_0402, symbol C
- added C?: 220nF 16V, Capacitors_SMD:C_0402, symbol C
- added C?: 22nF 16V, Capacitors_SMD:C_0402, symbol C
- added C? (x2): 470nF 6V3, Capacitors_SMD:C_0402, symbol C
- added C?: 1u 6V3, Capacitors_SMD:C_0402, symbol C
- added C?: 47u 16V, Capacitors_SMD:C_1206, symbol C
- added R? (x2): 20k, Resistors_SMD:R_0402, symbol R
- added R?: NM, Resistors_SMD:R_0402, symbol R
- added R?: 36k, Resistors_SMD:R_0402, symbol R
- added R?: 0R, Resistors_SMD:R_0402, symbol R
- added U?: DRV8886AT, lakotamm-motordriver:TSSOP-24_1E_4.4x7.8mm_Pitch0.65mm, symbol DRV8886AT
Connections:
- net ENA_2 is gone; now on net ENA: U6.18 (ENABLE)
- net nSLEEP_2 is gone; now on net nSLEEP: U6.17 (nSLEEP)
- net +3V3: now also R?.1
- net GND: now also C?.2, C?.2, C?.2, C?.2, C?.2, C?.2, R?.2, R?.2, U?.12 (GND), U?.25 (Thermal_pad), U?.6 (PGND), U?.9 (PGND)
- net VDD: now also C16.1, C18.1, C20.1, C23.1, C28.1, C30.1, C32.1, C34.1, U4.11 (VM), U4.4 (VM), U6.11 (VM), U6.4 (VM), C?.1, C?.1, C?.1, C?.1, U?.11 (VM), U?.4 (VM)
- net ENA_1 renamed ENA
- net ENA: now also U?.18 (ENABLE)
- net nSLEEP_1 renamed nSLEEP
- net nSLEEP: now also U?.17 (nSLEEP)
- new net: C?.1, U?.1 (CPL)
- new net: C?.1, U?.13 (AVDD)
- new net: C?.1, U?.14 (DVDD)
- new net: R?.1, U?.16 (RREF)
- new net: C?.2, U?.2 (CPH)
- new net: C?.2, U?.3 (VCP)
- new net: C?.1, R?.1, R?.2, R?.2
- new net DECAY_3: R?.1, R?.2, U?.24 (DECAY)
- new net DIR_3: U?.20 (DIR)
- new net M0_3: U?.21 (M0)
- new net M1_3: U?.22 (M1)
- new net MOT3_AOUT1: U?.5 (AOUT1)
- new net MOT3_AOUT2: U?.7 (AOUT2)
- new net MOT3_BOUT1: U?.10 (BOUT1)
- new net MOT3_BOUT2: U?.8 (BOUT2)
- new net RREF_3: R?.1
- new net STEP_3: U?.19 (STEP)
- new net TRQ_3: U?.23 (TRQ)
- new net nFAULT_3: U?.15 (nFAULT)
Other:
- moved on the sheet: C16, C17, C18, C19, C20, C22, C23, C24, C28, C29, C30, C31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
